Commit message: Cleanup and Update readme and robot files
Signed-off-by: Vatan Aksoy Tezer <vatanaksoytezer@gmail.com>

File: ros_ign_gazebo_demos/models/rrbot.urdf (robot description, URDF)
Before this commit: robot rrbot, 3 links, 2 joints
Links:
- added link base_link
Joints:
- added joint fixed_joint: type fixed, parent base_link, child link1, origin xyz=0 0 0 rpy=0 0 0
